File: openSX70-dongle_v2-9.sch (EAGLE design)
At the start: 22 parts

Commit message: Version 2.9 schematic
Other:
- note added: "2.9"
- note removed: "2.6"
Changed lines of the file:
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@@
 <plain>
 <text x="165.1" y="10.16" size="6.4516" layer="91">openSX70 dongle</text>
-<text x="244.856" y="-9.398" size="5.08" layer="97">2.6</text>
+<text x="244.856" y="-9.398" size="5.08" layer="97">2.9</text>
 </plain>
 <instances>
