File: openSX70-dongle_v3-2.sch (EAGLE design)
At the start: 24 parts

Commit message: New Gerbers, ready to order!
Other:
- note added: "3.2"
- note removed: "3.1"
Changed lines of the file:
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@@
 <plain>
 <text x="165.1" y="10.16" size="6.4516" layer="91">openSX70 dongle</text>
-<text x="244.856" y="-9.398" size="5.08" layer="97">3.1</text>
+<text x="244.856" y="-9.398" size="5.08" layer="97">3.2</text>
 </plain>
 <instances>
