File: openSX70-dongle-USB-V1.sch (EAGLE design)
At the start: 33 parts, among them J1 687106183722, U1 FT232RLSSOP

Commit message: dongle questions
Other:
- note added: "1.0"
- note added: "POWER FROM CAMERA (6V)"
- note added: "POWER FROM USB (5V)"
- note added: "openSX70 dongle-USB"
- note removed: "3.3"
- note removed: "openSX70 dongle"
Changed lines of the file:
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@@
 <sheet>
 <plain>
-<text x="165.1" y="10.16" size="6.4516" layer="91">openSX70 dongle</text>
-<text x="244.856" y="-9.398" size="5.08" layer="97">3.3</text>
+<text x="157.48" y="10.16" size="6.4516" layer="95">openSX70 dongle-USB</text>
+<text x="244.856" y="-9.398" size="5.08" layer="97">1.0</text>
+<text x="193.04" y="119.38" size="1.778" layer="91">POWER FROM CAMERA (6V)</text>
+<text x="66.04" y="160.02" size="1.778" layer="91">POWER FROM USB (5V)</text>
 </plain>
 <instances>
