File: openSX70-dongle-USB-V1-1.brd (EAGLE design)
At the start: 47.1 x 25.7 mm, 28 parts, among them J1 687106183722, U1 FT232RLSSOP

Commit message: ?
Parts:
- removed SW1, SW2: (no value), Seeed-Switch:SW5-2.0-8.8X4.4X4.7MM-90D
- removed TP+2.8V, TP_I/O: (no value), wirepad:SMD1,27-2,54
- added I/O, TP+3.3V, TP-GND: (no value), wirepad:SMD1,27-2,54
- added S2, S3: (no value), SparkFun-Switches:SWITCH_SPST_SMD_A
- moved S1 77.6 mm to (16.9, 43.5), flipped to the bottom
- moved J1 69.9 mm to (16.8, 42.7), turned to 180 degrees
- moved U$1 67.9 mm to (22.7, 1.14), turned to 90 degrees
- moved C3 60.4 mm to (11.6, 13.6)
- moved U1 50.2 mm to (18.7, 13.2), turned to 90 degrees
- moved C4 49.7 mm to (7.53, 14.6), turned to 270 degrees
- moved R6 44.8 mm to (24.9, 3.12), turned to 180 degrees
- moved R10 44.4 mm to (27.0, 3.12), turned to 180 degrees
- moved R1 34.3 mm to (3.59, 38.5), flipped to the top, turned to 180 degrees
- moved R5 27.3 mm to (4.82, 23.8), flipped to the top
- moved R3 26.2 mm to (8.82, 23.8), flipped to the top
- moved SELECTOR 24.4 mm to (23.1, 33.2), turned to 90 degrees
- moved DS2408 23.8 mm to (7.95, 31.3)
- moved PAD1 22.4 mm to (24.2, 34.5)
- moved USB1 21.1 mm to (17.2, 4.86)
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Connections:
- net 1W: now also I/O.1; no longer TP_I/O.1
- net 3V3OUT: now also S2.1, S3.1, TP+3.3V.1; no longer SW1.NC1, SW2.NC1, TP+2.8V.1
- net GND: now also TP-GND.1
- net N$6: now also S2.2; no longer SW2.COM
- net N$7: now also S3.2; no longer SW1.COM
Routing:
- net 5V: track 0.00 -> 87.9 mm, vias 0 -> 4
- net 3V3OUT: track 53.5 -> 136.3 mm, vias 0 -> 2
- net TXO: track 0.00 -> 53.3 mm, vias 0 -> 4
- net VCC-USB: track 0.00 -> 51.1 mm, vias 0 -> 4
- net RXI: track 0.00 -> 37.2 mm, vias 0 -> 2
- net DTR: track 0.00 -> 37.0 mm, vias 0 -> 2
- net N$7: track 14.3 -> 51.0 mm, vias 0 -> 3
- net N$13: track 27.2 -> 63.6 mm
- net N$3: track 26.1 -> 54.6 mm, vias 1 -> 3
- net TXLED: track 0.00 -> 15.4 mm, vias 0 -> 2
- net RXLED: track 0.00 -> 15.0 mm, vias 0 -> 2
- net USB_D+: track 0.00 -> 14.4 mm
- net N$16: track 0.00 -> 13.7 mm
- net N$8: track 15.1 -> 3.55 mm, vias 1 -> 0
- net N$11: track 21.4 -> 14.8 mm, vias 1 -> 0
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Other:
- board size 47.1 x 25.7 mm -> 29 x 45 mm
- board text added: "openSX70"
- board text removed: "+"
- board text removed: "1-W"
- board text removed: "2.8V"
- board text removed: "20181009 v.3.7"
- board text removed: "6V"
- board text removed: "CE"
- board text removed: "GND"
- board text removed: "N/C"
- board text removed: "OPTION SELECTOR"
- board text removed: "PC-FLASH"
- board text removed: "S1"
- board text removed: "S2"
- board text removed: "VCC"
- board text removed: "bottom"
- board text removed: "openSX70 dongle 3.7"
- board text removed: "top"
- board text removed: "www.openSX70.com"
