File: openSX70-dongle-USB-V1-1.sch (EAGLE design)
At the start: 28 parts, among them J1 687106183722, U1 FT232RLSSOP

Commit message: ?
Parts:
- removed SW1, SW2: (no value), Seeed-Switch:DIP-TOGGLE-SWITCH-ON-ON(3+2P-8.8X4.6MM)-90D
- added S2, S3: (no value), SparkFun-Switches:SWITCH-SPDT-SMD-RIGHT-ANGLE
- added TP-GND: (no value), wirepad:SMD2
- renumbered TP+2.8V to TP+3.3V, TP_I/O to I/O
Connections:
- net 3V3OUT: now also S2.O, S3.O; no longer SW1.NC1, SW2.NC1
- net GND: now also TP-GND.P
- net N$6: now also S2.P; no longer SW2.COM
- net N$7: now also S3.P; no longer SW1.COM
Changed lines of the file:
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@@
 </variantdefs>
 <classes>
-<class number="0" name="GND" width="0.3048" drill="0">
+<class number="0" name="GND" width="0.2032" drill="0">
 </class>
-<class number="1" name="power" width="0.254" drill="0">
+<class number="1" name="power" width="0.2032" drill="0">
 </class>
-<class number="2" name="2.8V" width="0.254" drill="0">
+<class number="2" name="2.8V" width="0.2032" drill="0">
 </class>
 </classes>
@@
 <part name="PC-FLASH" library="SparkFun-Connectors" deviceset="AUDIO_JACK_3.5MM" device="_PTH"/>
 <part name="FRAME1" library="frames" library_urn="urn:adsk.eagle:library:229" deviceset="DINA4_L" device=""/>
-<part name="TP+2.8V" library="wirepad" library_urn="urn:adsk.eagle:library:412" deviceset="SMD2" device="" package3d_urn="urn:adsk.eagle:package:30839/1"/>
-<part name="TP_I/O" library="wirepad" library_urn="urn:adsk.eagle:library:412" deviceset="SMD2" device="" package3d_urn="urn:adsk.eagle:package:30839/1"/>
+<part name="TP+3.3V" library="wirepad" library_urn="urn:adsk.eagle:library:412" deviceset="SMD2" device="" package3d_urn="urn:adsk.eagle:package:30839/1"/>
+<part name="I/O" library="wirepad" library_urn="urn:adsk.eagle:library:412" deviceset="SMD2" device="" package3d_urn="urn:adsk.eagle:package:30839/1"/>
 <part name="GND-ISO6" library="supply2" library_urn="urn:adsk.eagle:library:372" deviceset="GND" device=""/>
 <part name="GND-ISO11" library="supply2" library_urn="urn:adsk.eagle:library:372" deviceset="GND" device=""/>
 <part name="GND-ISO12" library="supply2" library_urn="urn:adsk.eagle:library:372" deviceset="GND" device=""/>
-<part name="SW1" library="Seeed-Switch" deviceset="DIP-TOGGLE-SWITCH-ON-ON(3+2P-8.8X4.6MM)-90D" device=""/>
-<part name="SW2" library="Seeed-Switch" deviceset="DIP-TOGGLE-SWITCH-ON-ON(3+2P-8.8X4.6MM)-90D" device=""/>
 <part name="PAD1" library="wirepad" library_urn="urn:adsk.eagle:library:412" deviceset="WIREPAD" device="1,6/0,8" package3d_urn="urn:adsk.eagle:package:30830/1"/>
 <part name="C3" library="openSX70_PATHFINDER_V5.5-SEEED_20180522" deviceset="CERAMIC-100NF-50V-10%-X7R(0603)" device="" value="100nf"/>
@@
 <part name="S1" library="SparkFun-Switches" library_urn="urn:adsk.eagle:library:535" deviceset="SWITCH-SPDT" device="-SMD-RIGHT-ANGLE" package3d_urn="urn:adsk.eagle:package:40179/1"/>
 <part name="U$1" library="_openSX70" deviceset="DUAL-LED-0603-BIS" device=""/>
+<part name="GND-ISO2" library="supply2" library_urn="urn:adsk.eagle:library:372" deviceset="GND" device=""/>
+<part name="S2" library="SparkFun-Switches" library_urn="urn:adsk.eagle:library:535" deviceset="SWITCH-SPDT" device="-SMD-RIGHT-ANGLE" package3d_urn="urn:adsk.eagle:package:40179/1"/>
+<part name="S3" library="SparkFun-Switches" library_urn="urn:adsk.eagle:library:535" deviceset="SWITCH-SPDT" device="-SMD-RIGHT-ANGLE" package3d_urn="urn:adsk.eagle:package:40179/1"/>
+<part name="TP-GND" library="wirepad" library_urn="urn:adsk.eagle:library:412" deviceset="SMD2" device="" package3d_urn="urn:adsk.eagle:package:30839/1"/>
 </parts>
 <sheets>
@@
 <attribute name="DRAWING_NAME" x="172.72" y="3.81" size="2.54" layer="94"/>
 </instance>
-<instance part="TP+2.8V" gate="1" x="55.88" y="60.96" rot="R270">
+<instance part="TP+3.3V" gate="1" x="55.88" y="60.96" rot="R270">
 <attribute name="NAME" x="57.7342" y="62.103" size="1.778" layer="95" rot="R270"/>
 <attribute name="VALUE" x="52.578" y="62.103" size="1.778" layer="96" rot="R270"/>
 </instance>
-<instance part="TP_I/O" gate="1" x="55.88" y="50.8" rot="R270">
+<instance part="I/O" gate="1" x="55.88" y="50.8" rot="R270">
 <attribute name="NAME" x="57.7342" y="51.943" size="1.778" layer="95" rot="R270"/>
 <attribute name="VALUE" x="52.578" y="51.943" size="1.778" layer="96" rot="R270"/>
@@
 <instance part="GND-ISO12" gate="GND" x="185.42" y="66.04" rot="R90">
 <attribute name="VALUE" x="188.595" y="64.135" size="1.778" layer="96" rot="R90"/>
-</instance>
-<instance part="SW1" gate="G$1" x="144.78" y="10.16">
-<attribute name="NAME" x="140.97" y="16.51" size="1.27" layer="95" ratio="10"/>
-<attribute name="VALUE" x="140.97" y="2.54" size="1.27" layer="96" ratio="10"/>
-</instance>
-<instance part="SW2" gate="G$1" x="144.78" y="30.48">
-<attribute name="NAME" x="140.97" y="36.83" size="1.27" layer="95" ratio="10"/>
-<attribute name="VALUE" x="140.97" y="22.86" size="1.27" layer="96" ratio="10"/>
 </instance>
 <instance part="PAD1" gate="G$1" x="114.3" y="104.14" rot="R180">
@@
 <attribute name="NAME" x="178.816" y="130.048" size="1.778" layer="95" rot="R90"/>
 <attribute name="NAME" x="186.436" y="130.048" size="1.778" layer="95" rot="R90"/>
+</instance>
+<instance part="GND-ISO2" gate="GND" x="7.62" y="25.4" rot="R270">
+<attribute name="VALUE" x="4.445" y="27.305" size="1.778" layer="96" rot="R270"/>
+</instance>
+<instance part="S2" gate="1" x="142.24" y="30.48">
+<attribute name="NAME" x="143.51" y="33.528" size="1.778" layer="95" font="vector" align="bottom-center"/>
+<attribute name="VALUE" x="143.256" y="27.178" size="1.778" layer="96" font="vector" align="top-center"/>
+</instance>
+<instance part="S3" gate="1" x="137.16" y="10.16">
+<attribute name="NAME" x="138.43" y="13.208" size="1.778" layer="95" font="vector" align="bottom-center"/>
+<attribute name="VALUE" x="138.176" y="6.858" size="1.778" layer="96" font="vector" align="top-center"/>
+</instance>
+<instance part="TP-GND" gate="1" x="66.04" y="40.64" rot="R270">
+<attribute name="NAME" x="67.8942" y="41.783" size="1.778" layer="95" rot="R270"/>
+<attribute name="VALUE" x="62.738" y="41.783" size="1.778" layer="96" rot="R270"/>
 </instance>
 </instances>
@@
 <wire x1="45.72" y1="33.02" x2="45.72" y2="30.48" width="0.1524" layer="91"/>
 <junction x="45.72" y="30.48"/>
-<pinref part="TP_I/O" gate="1" pin="P"/>
+<pinref part="I/O" gate="1" pin="P"/>
 <wire x1="55.88" y1="48.26" x2="55.88" y2="45.72" width="0.1524" layer="91"/>
 <junction x="55.88" y="45.72"/>
@@
 <wire x1="129.54" y1="30.48" x2="134.62" y2="30.48" width="0.1524" layer="91"/>
 <junction x="129.54" y="30.48"/>
-<pinref part="SW2" gate="G$1" pin="COM"/>
 <wire x1="135.89" y1="30.48" x2="129.54" y2="30.48" width="0.1524" layer="91"/>
+<pinref part="S2" gate="1" pin="P"/>
+<wire x1="139.7" y1="30.48" x2="129.54" y2="30.48" width="0.1524" layer="91"/>
 </segment>
 </net>
@@
 <wire x1="116.84" y1="10.16" x2="121.92" y2="10.16" width="0.1524" layer="91"/>
 <junction x="116.84" y="10.16"/>
-<pinref part="SW1" gate="G$1" pin="COM"/>
-<wire x1="135.89" y1="10.16" x2="116.84" y2="10.16" width="0.1524" layer="91"/>
+<wire x1="135.89" y1="10.16" x2="134.62" y2="10.16" width="0.1524" layer="91"/>
+<pinref part="S3" gate="1" pin="P"/>
+<wire x1="134.62" y1="10.16" x2="116.84" y2="10.16" width="0.1524" layer="91"/>
+<junction x="134.62" y="10.16"/>
 </segment>
 </net>
@@
 <wire x1="66.04" y1="38.1" x2="71.12" y2="38.1" width="0.1524" layer="91"/>
 <wire x1="58.42" y1="25.4" x2="58.42" y2="38.1" width="0.1524" layer="91"/>
-<wire x1="5.08" y1="25.4" x2="58.42" y2="25.4" width="0.1524" layer="91"/>
 <pinref part="GND-ISO1" gate="GND" pin="GND"/>
+<wire x1="10.16" y1="25.4" x2="58.42" y2="25.4" width="0.1524" layer="91"/>
 <wire x1="66.04" y1="35.56" x2="66.04" y2="38.1" width="0.1524" layer="91"/>
 <junction x="66.04" y="38.1"/>
+<label x="15.24" y="27.94" size="1.778" layer="95"/>
+<pinref part="GND-ISO2" gate="GND" pin="GND"/>
+<pinref part="TP-GND" gate="1" pin="P"/>
 </segment>
 <segment>
@@
 <wire x1="91.44" y1="22.86" x2="111.76" y2="22.86" width="0.1524" layer="91"/>
 <junction x="71.12" y="53.34"/>
-<pinref part="TP+2.8V" gate="1" pin="P"/>
+<pinref part="TP+3.3V" gate="1" pin="P"/>
 <wire x1="55.88" y1="53.34" x2="71.12" y2="53.34" width="0.1524" layer="91"/>
 <wire x1="55.88" y1="58.42" x2="55.88" y2="53.34" width="0.1524" layer="91"/>
@@
 </segment>
 <segment>
-<pinref part="SW2" gate="G$1" pin="NC1"/>
-<wire x1="135.89" y1="35.56" x2="124.46" y2="35.56" width="0.1524" layer="91"/>
-<label x="124.46" y="33.02" size="1.778" layer="95"/>
-</segment>
-<segment>
-<pinref part="SW1" gate="G$1" pin="NC1"/>
-<wire x1="135.89" y1="15.24" x2="121.92" y2="15.24" width="0.1524" layer="91"/>
-<label x="121.92" y="17.78" size="1.778" layer="95"/>
+<wire x1="156.21" y1="33.02" x2="147.32" y2="33.02" width="0.1524" layer="91"/>
+<label x="157.48" y="33.02" size="1.778" layer="95"/>
+<pinref part="S2" gate="1" pin="O"/>
+<wire x1="147.32" y1="33.02" x2="144.78" y2="33.02" width="0.1524" layer="91"/>
+<junction x="147.32" y="33.02"/>
 </segment>
 <segment>
@@
 <label x="43.18" y="0" size="1.778" layer="95" rot="R180"/>
 </segment>
-</net>
+<segment>
+<pinref part="S3" gate="1" pin="O"/>
+<wire x1="142.24" y1="12.7" x2="149.86" y2="12.7" width="0.1524" layer="91"/>
+<label x="142.24" y="15.24" size="1.778" layer="95"/>
+</segment>
+</net>
