File: openSX70-dongle_v3-7.sch (EAGLE design)
At the start: 25 parts

Commit message: 3.7 gerbers
Parts:
- renumbered LED1 to LED
Changed lines of the file:
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@@
 <part name="GND-ISO1" library="supply2" library_urn="urn:adsk.eagle:library:372" deviceset="GND" device=""/>
 <part name="GND-ISO8" library="supply2" library_urn="urn:adsk.eagle:library:372" deviceset="GND" device=""/>
-<part name="LED1" library="adafruit" library_urn="urn:adsk.eagle:library:420" deviceset="LED" device="3MM"/>
+<part name="LED" library="adafruit" library_urn="urn:adsk.eagle:library:420" deviceset="LED" device="3MM"/>
 <part name="OPTO" library="openSX70" deviceset="TLP127" device="" value="TLP127"/>
 <part name="R12" library="rcl" library_urn="urn:adsk.eagle:library:334" deviceset="R-US_" device="M0805" package3d_urn="urn:adsk.eagle:package:23556/1" value="220R"/>
@@
 <attribute name="VALUE" x="196.215" y="56.515" size="1.778" layer="96" rot="R90"/>
 </instance>
-<instance part="LED1" gate="G$1" x="91.44" y="35.56" rot="MR270">
+<instance part="LED" gate="G$1" x="91.44" y="35.56" rot="MR270">
 <attribute name="NAME" x="96.012" y="32.004" size="1.778" layer="95" rot="MR0"/>
 <attribute name="VALUE" x="96.012" y="29.845" size="1.778" layer="96" rot="MR0"/>
@@
 <net name="N$2" class="0">
 <segment>
-<pinref part="LED1" gate="G$1" pin="C"/>
+<pinref part="LED" gate="G$1" pin="C"/>
 <pinref part="R9" gate="G$1" pin="2"/>
 </segment>
@@
 </segment>
 <segment>
-<pinref part="LED1" gate="G$1" pin="A"/>
+<pinref part="LED" gate="G$1" pin="A"/>
 <wire x1="86.36" y1="35.56" x2="88.9" y2="35.56" width="0.1524" layer="91"/>
 <label x="86.36" y="38.1" size="1.778" layer="95" rot="R180"/>
