File: openSX70-dongle_v3-8.brd (EAGLE design)
At the start: 47.1 x 25.7 mm, 28 parts, among them J1 687106183722, U1 FT232RLSSOP

Commit message: ?
Parts:
- removed C3: 100nf, openSX70_PATHFINDER_V5.5-SEEED_20180522:C0603
- removed C4: 10uf, Seeed-Capacitor-2016:AVX-A
- removed J1: 687106183722, openSX70_PATHFINDER_V5.5-SEEED_20180522:687106183722
- removed R10, R6: 1K, openSX70_PATHFINDER_V5.5-SEEED_20180522:R0603
- removed S1: (no value), SparkFun-Switches:SWITCH_SPST_SMD_A
- removed U1: FT232RLSSOP, SparkFun:SSOP28DB
- removed USB1: 10118193-0001LF, Seeed-Connector -2016:MICRO-USB5+6P-SMD-0.65-B
- added C1, C2: 1.0uF, rcl:C0603
- added REG: NCP4688, openSX70:SOT-23-5
- added TP+6V, TP-: (no value), wirepad:SMD1,27-2,54
- U$1: value DUAL-LED-0603-BIS -> FLASH-EDGE-CONNECTOR; device _openSX70:LED_APHB1608SYKSURKC -> SX70-flash:FLASH-EDGE-8
- moved U$1 71.3 mm to (25.7, 3.06)
- moved R3 0.22 mm to (34.2, 17.4)
- moved R8 0.22 mm to (19.2, 17.4)
- moved R7 0.13 mm to (22.2, 17.4)
- moved R2 0.09 mm to (25.2, 17.4)
- moved R9 0.08 mm to (17.6, 11.0)
- moved R12 0.08 mm to (17.6, 13.6)
- moved R5 0.08 mm to (31.4, 17.4)
- moved R4 0.06 mm to (28.3, 17.4)
Connections:
- removed net 1W: DS2408.4, J1.2, R1.1, TP_I/O.1
- removed net 3V3OUT: DS2408.10, DS2408.3, LED.A, OPTO.1, PAD1.1, R1.2, SELECTOR.C, SW1.NC1, SW2.NC1, TP+2.8V.1, U1.17
- removed net 5V: C3.1, C4.+, R10.2, R6.2, S1.1, U1.20, U1.4
- removed net 5V-J1: J1.3, S1.2
- removed net CTS: U1.11
- removed net DTR: J1.6, U1.2
- removed net N$14: R10.1, U$1.3
- removed net N$16: U1.16, USB1.2
- removed net N$9: R6.1, U$1.1
- removed net RXI: J1.5, U1.5
- removed net RXLED: U$1.4, U1.22
- removed net TXLED: U$1.2, U1.23
- removed net TXO: J1.4, U1.1
- removed net USB_D+: U1.15, USB1.3
- removed net VCC-USB: S1.3, USB1.1
- new net 2.8V: C2.1, DS2408.10, DS2408.3, LED.A, OPTO.1, PAD1.1, R1.2, REG.5, SELECTOR.C, SW1.NC1, SW2.NC1, TP+2.8V.1
- new net N$1: DS2408.4, R1.1, TP_I/O.1, U$1.P$2
- new net VCC: C1.1, REG.1, REG.3, TP+6V.1, U$1.P$6
- net GND: now also C1.2, C2.2, REG.2, TP-.1, U$1.P$1; no longer C3.2, C4.-, J1.1, U1.18, U1.21, U1.25, U1.26, U1.7, USB1.5, USB1.S1, USB1.S2, USB1.S3, USB1.S4, USB1.S5, USB1.S6
Routing:
- net 2.8V: track 0.00 -> 93.9 mm, vias 0 -> 1
- net 3V3OUT: track 53.5 -> 0.00 mm
- net N$1: track 0.00 -> 38.8 mm, vias 0 -> 1
- net 1W: track 35.7 -> 0.00 mm, vias 1 -> 0
- net VCC: track 0.00 -> 25.0 mm, vias 0 -> 1
- net GND: track 0.00 -> 4.10 mm
Other:
- board text added: "20181106 v.3.8"
- board text removed: "20181009 v.3.7"
