File: openSX70-dongle_v3-8.sch (EAGLE design)
At the start: 28 parts, among them J1 687106183722, U1 FT232RLSSOP

Commit message: ?
Parts:
- removed C3: 100nf, openSX70_PATHFINDER_V5.5-SEEED_20180522:CERAMIC-100NF-50V-10%-X7R(0603)
- removed C4: 10uf, Seeed-Capacitor-2016:TANTALUM-SMD-10UF-16V-10%(AVX-A)
- removed J1: 687106183722, openSX70_PATHFINDER_V5.5-SEEED_20180522:687106183722
- removed R10, R6: 1K, openSX70_PATHFINDER_V5.5-SEEED_20180522:SMD-RES-1K-1%-1/10W(0603)
- removed S1: (no value), SparkFun-Switches:SWITCH-SPDT-SMD-RIGHT-ANGLE
- removed U1: FT232RLSSOP, SparkFun:FT232RLSSOP
- removed USB1: 10118193-0001LF, Seeed-Connector -2016:MICRO-USB-SMD-B-(10118193-0001LF)
- added C1, C2: 1.0uF, rcl:C-EUC0603
- added REG: NCP4688, openSX70:NCP4688
- added TP+6V, TP-: (no value), wirepad:SMD2
- U$1: value DUAL-LED-0603-BIS -> FLASH-EDGE-CONNECTOR; device _openSX70:DUAL-LED-0603-BIS -> SX70-flash:FLASH-EDGE-CONNECTOR
Connections:
- removed net 1W: DS2408.I/O, J1.5, R1.1, TP_I/O.P
- removed net 3V3OUT: DS2408.RSTZ, DS2408.VCC, LED.A, OPTO.A, PAD1.P, R1.2, SELECTOR.C, SW1.NC1, SW2.NC1, TP+2.8V.P, U1.3V3OUT
- removed net 5V: C3.1, C4.+, R10.2, R6.2, S1.O, U1.VCC, U1.VCCIO
- removed net 5V-J1: J1.4, S1.P
- removed net CTS: U1.CTS
- removed net DTR: J1.1, U1.DTR
- removed net N$14: R10.1, U$1.A1
- removed net N$16: U1.USBDM, USB1.DM
- removed net N$9: R6.1, U$1.A
- removed net RXI: J1.2, U1.RXD
- removed net RXLED: U$1.C1, U1.RXLED
- removed net TXLED: U$1.C, U1.TXLED
- removed net TXO: J1.3, U1.TXD
- removed net USB_D+: U1.USBDP, USB1.DP
- removed net VCC-USB: S1.S, USB1.VCC
- new net 2.8V: C2.1, DS2408.RSTZ, DS2408.VCC, LED.A, OPTO.A, PAD1.P, R1.2, REG.VOUT, SELECTOR.C, SW1.NC1, SW2.NC1, TP+2.8V.P
- new net N$1: DS2408.I/O, R1.1, TP_I/O.P, U$1.S2
- new net VCC: C1.1, REG.CE, REG.VIN, TP+6V.P, U$1.VCC
- net GND: now also C1.2, C2.2, REG.GND, TP-.P, U$1.GND; no longer C3.2, C4.-, J1.6, U1.AGND, U1.GND18, U1.GND21, U1.GND7, U1.TEST, USB1.GND@1, USB1.GND@2, USB1.GND@3, USB1.GND@4, USB1.GND@5
Other:
- note added: "3.3"
- note added: "openSX70 dongle"
- note removed: "1.0"
- note removed: "POWER FROM CAMERA (6V)"
- note removed: "POWER FROM USB (5V)"
- note removed: "openSX70 dongle-USB"
- moved on the sheet: LED, OPTO, PAD1, PC-FLASH, R1, R12, R2, R3, R4, R5, R7, R8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
