File: openSX70-dongle_SEEED_v51.brd (EAGLE design)
At the start: 94 x 43.9 mm, 24 parts, among them SW1 MK-12C02 G1.5, SW2 MK-12C02 G1.5, X1 1503_02

Commit message: no message
Parts:
- added 1-WIRE, 1-WIRE-H, 2.8V-H, 2.8V-V, GND, GND-H, LED-H, S1-H, S1-V, S2-H, S2-V, VCC, VCC-H: SX70-S-PAD-NEW, openSX70:SX70-S-PAD2
Connections:
- removed net GND: C1.2, C2.2, DS2408.5, R2.2, R3.1, R4.1, R5.1, R7.2, R8.2, REG.2, TP-.1, U$1.P$1
- removed net N$1: DS2408.4, R1.1, TP_I/O.1, U$1.P$2
- removed net N$6: DS2408.11, R8.1, SW2.COM
- removed net N$7: DS2408.9, R7.1, SW1.COM
- removed net N$8: DS2408.8, R9.1
- removed net VCC: C1.1, REG.1, REG.3, TP+6V.1, U$1.P$6
- new net 1-WIRE-H: 1-WIRE-H.P$1, DS2408.4, R1.1, TP_I/O.1
- new net 1-WIRE-V: 1-WIRE.P$1, U$1.P$2
- new net 2.8V-H: 2.8V-H.P$1, C2.1, DS2408.10, DS2408.3, R1.2, REG.5, TP+2.8V.1
- new net 2.8V-V: 2.8V-V.P$1, LED1.A, SW1.A, SW2.A
- new net GND-H: C1.2, C2.2, DS2408.5, GND-H.P$1, R2.2, R3.1, R4.1, R5.1, REG.2, TP-.1
- new net GND-V: GND.P$1, R7.2, R8.2, U$1.P$1
- new net LED-H: DS2408.8, LED-H.P$1
- new net LED-V: R9.1
- new net S1-H: DS2408.9, S1-H.P$1
- new net S1-V: R7.1, S1-V.P$1, SW1.COM
- new net S2-H: DS2408.11, S2-H.P$1
- new net S2-V: R8.1, S2-V.P$1, SW2.COM
- new net VCC-H: C1.1, REG.1, REG.3, TP+6V.1, VCC-H.P$1
- new net VCC-V: U$1.P$6, VCC.P$1
- net 2.8V: no longer C2.1, DS2408.10, DS2408.3, LED1.A, R1.2, REG.5, SW1.A, SW2.A, TP+2.8V.1

Commit message: new origami design
Parts:
- SELECTOR: value CTS221AMX16 -> SELECTOR-4-1-SMD-A6RS; device openSX70:CTS221AMX16 -> _openSX70:A6RS-161RS
- X1: value 1503_02 -> JACK-SMD-SJ-3523-SMT-TR; device con-lumberg:1503_02 -> _openSX70:CUI_SJ-3523-SMT-TR
- moved R2 24.8 mm to (53.7, 41.1)
- moved R4 24.6 mm to (56.3, 33.8), turned to 90 degrees
- moved R8 23.2 mm to (56.4, 37.1)
- moved C2 9.42 mm to (33.0, 34.2)
- moved C1 8.90 mm to (21.9, 34.1), turned to 270 degrees
- moved REG 8.29 mm to (27.9, 34.1)
- moved SELECTOR 7.11 mm to (68.2, 33.3), turned to 90 degrees
- moved LED1 4.70 mm to (11.2, 10.4)
- moved R3 3.95 mm to (39.8, 41.7), turned to 0 degrees
- moved X1 2.12 mm to (-18.7, 39.4), turned to 0 degrees
- moved OPTO 1.35 mm to (-3.03, 41.7)
Connections:
- net 2.8V: no longer SELECTOR.C2
