File: openSX70-dongle_SEEED_v52.brd (EAGLE design)
At the start: 94 x 43.9 mm, 25 parts, among them SW1 MK-12C02 G1.5, SW2 MK-12C02 G1.5, X1 JACK-SMD-SJ-3523-SMT-TR

Commit message: WIP origami
Parts:
- added U$1: FLASH-BRIDGE-SW1-SW2-LED-SMALL, _openSX70:FLASH-8-BRIDGE-SW1-SW2-LED-SMALL
- added U$4: FLASH-BRIDGE-SMALL, _openSX70:FLASH-8-BRIDGE1-SMALL
Changed lines of the file:
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@@
 <element name="R1" library="Seeed-Resistor" library_urn="urn:adsk.eagle:library:474" package="R0603" package3d_urn="urn:adsk.eagle:package:32791/1" value="4.7K" x="34.2496" y="42.7934" rot="R270">
 <attribute name="MPN" value="RC0603JR-074K7L" x="34.2496" y="42.7934" size="1.778" layer="27" rot="R270" display="off"/>
-<attribute name="NAME" x="33.7035" y="44.673" size="0.8128" layer="25" font="vector"/>
+<attribute name="NAME" x="33.4035" y="43.773" size="0.8128" layer="25" font="vector"/>
 <attribute name="VALUE" value="4.7K" x="31.7096" y="44.0634" size="0.8128" layer="27" font="vector" rot="R270"/>
 </element>
@@
 </element>
 <element name="TP-" library="wirepad" library_urn="urn:adsk.eagle:library:412" package="SMD1,27-2,54" package3d_urn="urn:adsk.eagle:package:30839/1" value="" x="21.7271" y="44.1216" rot="R90">
-<attribute name="NAME" x="24.2414" y="45.8235" size="0.8128" layer="25" font="vector" rot="R180"/>
+<attribute name="NAME" x="22.7414" y="43.1235" size="0.8128" layer="25" font="vector" rot="R180"/>
 <attribute name="VALUE" x="21.7271" y="44.1216" size="0.0254" layer="27" rot="R90"/>
 </element>
 <element name="TP_I/O" library="wirepad" library_urn="urn:adsk.eagle:library:412" package="SMD1,27-2,54" package3d_urn="urn:adsk.eagle:package:30839/1" value="" x="28.2509" y="44.1563" rot="R90">
-<attribute name="NAME" x="30.943" y="45.6931" size="0.8128" layer="25" font="vector" rot="R180"/>
+<attribute name="NAME" x="30.043" y="43.1931" size="0.8128" layer="25" font="vector" rot="R180"/>
 <attribute name="VALUE" x="28.2509" y="44.1563" size="0.0254" layer="27" rot="R90"/>
 </element>
@@
 </element>
 <element name="TP+6V" library="wirepad" library_urn="urn:adsk.eagle:library:412" package="SMD1,27-2,54" package3d_urn="urn:adsk.eagle:package:30839/1" value="" x="17.889" y="44.198" rot="R90">
-<attribute name="NAME" x="20.3906" y="45.8364" size="0.8128" layer="25" font="vector" rot="R180"/>
+<attribute name="NAME" x="19.2906" y="43.0364" size="0.8128" layer="25" font="vector" rot="R180"/>
 <attribute name="VALUE" x="17.889" y="44.198" size="0.0254" layer="27" rot="R90"/>
 </element>
@@
 <attribute name="NAME" x="14.64" y="35.01" size="1.778" layer="21" font="vector"/>
 </element>
+<element name="U$1" library="_openSX70" package="FLASH-8-BRIDGE-SW1-SW2-LED-SMALL" value="FLASH-BRIDGE-SW1-SW2-LED-SMALL" x="26.2" y="15.7">
+<attribute name="NAME" x="7.54" y="23.21" size="1.778" layer="21" font="vector"/>
+</element>
+<element name="U$4" library="_openSX70" package="FLASH-8-BRIDGE1-SMALL" value="FLASH-BRIDGE-SMALL" x="-6.9" y="-1.8">
+<attribute name="NAME" x="-17.06" y="2.01" size="1.778" layer="21" font="vector"/>
+</element>
 </elements>
