File: openSX70-dongle_SEEED_v52.sch (EAGLE design)
At the start: 25 parts, among them SW1 MK-12C02 G1.5, SW2 MK-12C02 G1.5, X1 JACK-SMD-SJ-3523-SMT-TR

Commit message: WIP origami
Parts:
- added U$1: FLASH-BRIDGE-SW1-SW2-LED-SMALL, _openSX70:FLASH-BRIDGE-SW1-SW2-LED-SMALL
- added U$4: FLASH-BRIDGE-SMALL, _openSX70:FLASH-BRIDGE-SMALL
Changed lines of the file:
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@@
 <part name="U$2" library="_openSX70" deviceset="FLASH-BRIDGE1" device=""/>
 <part name="U$3" library="_openSX70" deviceset="FLASH-BRIDGE-SW1-SW2-LED" device=""/>
+<part name="U$1" library="_openSX70" deviceset="FLASH-BRIDGE-SW1-SW2-LED-SMALL" device=""/>
+<part name="U$4" library="_openSX70" deviceset="FLASH-BRIDGE-SMALL" device=""/>
 </parts>
 <sheets>
@@
 <instance part="U$2" gate="G$1" x="86.36" y="55.88"/>
 <instance part="U$3" gate="G$1" x="83.82" y="12.7"/>
+<instance part="U$1" gate="G$1" x="83.82" y="114.3"/>
+<instance part="U$4" gate="G$1" x="86.36" y="93.98"/>
 </instances>
 <busses>
