File: 20190105_ORIGAMI_V1-H-08slot.brd (EAGLE design)
At the start: 94 x 13 mm, 21 parts, among them X1 JACK-SMD-SJ-3523-SMT-TR

Commit message: chanmges
Parts:
- DS2408: device DS2408-joaco:SO16 -> _openSX70:SO16
- OPTO: device openSX70:SO-4 -> _openSX70:SO-4
Changed lines of the file:
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@@
 <drawing>
 <settings>
-<setting alwaysvectorfont="no"/>
+<setting alwaysvectorfont="yes"/>
 <setting verticaltext="up"/>
 </settings>
@@
 </layers>
 <board>
+<fusionsync huburn="a.cGVyc29uYWw6dWUyYjc0YWI4" projecturn="a.cGVyc29uYWw6dWUyYjc0YWI4IzIwMTcwNzE4ODQ1NjQxNTE" f3durn="urn:adsk.wipprod:dm.lineage:AoAC12g0SkmPLSMk-iGgLg" pcbguid="edb3502e-7c8f-4c82-9d71-33b41b792465" lastpulledtime="" lastsyncedchangeguid="dac62d5c-c7c7-73c4-919d-cd9f57cf9c74"/>
 <plain>
 <text x="53.024" y="11.4764" size="1.27" layer="21" font="vector" rot="R180">20190106_ORIGAMI_V1.1-0.9mm</text>
@@
 </autorouter>
 <elements>
-<element name="DS2408" library="DS2408-joaco" package="SO16" value="DS2408" x="68.7944" y="6.7162" rot="R90">
+<element name="DS2408" library="_openSX70" library_urn="urn:adsk.eagle:library:7902803" package="SO16" package3d_urn="urn:adsk.eagle:package:7902916/2" value="DS2408" x="68.7944" y="6.7162" rot="R90">
 <attribute name="NAME" x="69.1404" y="8.3482" size="0.8128" layer="25" font="vector" ratio="10" rot="R270"/>
 <attribute name="VALUE" x="69.4294" y="2.6522" size="0.8128" layer="27" font="vector" ratio="10" rot="R90"/>
@@
 <attribute name="VALUE" value="Yellow" x="9.7088" y="0.15" size="1.27" layer="27" ratio="10"/>
 </element>
-<element name="OPTO" library="openSX70" package="SO-4" value="TLP127" x="21.1746" y="10.2208" rot="R180">
+<element name="OPTO" library="_openSX70" library_urn="urn:adsk.eagle:library:7902803" package="SO-4" package3d_urn="urn:adsk.eagle:package:7902924/3" value="TLP127" x="21.1746" y="10.2208" rot="R180">
 <attribute name="NAME" x="22.4446" y="11.4908" size="0.8128" layer="25" font="vector" rot="R180"/>
 <attribute name="VALUE" x="23.0796" y="14.6658" size="1.27" layer="27" rot="R180"/>
@@
 <attribute name="VALUE" value="220R" x="59.0031" y="3.1322" size="1.27" layer="27" font="vector" rot="R270"/>
 </element>
-<element name="SELECTOR" library="_openSX70" package="A6RS-161RS" value="SELECTOR-4-1-SMD-A6RS" x="88.75" y="1.785" rot="R90">
+<element name="SELECTOR" library="_openSX70" library_urn="urn:adsk.eagle:library:7902803" package="A6RS-161RS" package3d_urn="urn:adsk.eagle:package:7902943/4" value="SELECTOR-4-1-SMD-A6RS" x="88.75" y="1.785" rot="R90">
 <attribute name="NAME" x="91.3535" y="8.008" size="0.8128" layer="25" font="vector" ratio="10" rot="R180"/>
 <attribute name="VALUE" x="96.116" y="-3.295" size="1.778" layer="27" ratio="10" rot="R90"/>
@@
 <attribute name="VALUE" value="1uf" x="30.0396" y="1.2262" size="0.6096" layer="27" rot="R90"/>
 </element>
-<element name="X1" library="_openSX70" package="CUI_SJ-3523-SMT-TR" value="JACK-SMD-SJ-3523-SMT-TR" x="4.76" y="6.9">
+<element name="X1" library="_openSX70" library_urn="urn:adsk.eagle:library:7902803" package="CUI_SJ-3523-SMT-TR" package3d_urn="urn:adsk.eagle:package:7902944/3" value="JACK-SMD-SJ-3523-SMT-TR" x="4.76" y="6.9">
 <attribute name="AVAILABILITY" value="Unavailable" x="4.76" y="6.9" size="1.778" layer="27" display="off"/>
 <attribute name="CUI_PURCHASE_URL" value="https://www.cui.com/product/interconnect/audio-connectors/3.5-mm-jacks/sj-352x-smt-series?utm_source=snapeda.com&amp;utm_medium=referral&amp;utm_campaign=snapedaBOM" x="4.76" y="6.9" size="1.778" layer="27" display="off"/>
@@
 <attribute name="VALUE" x="11.11" y="-3.26" size="1.27" layer="27" rot="R90"/>
 </element>
-<element name="U$2" library="_openSX70" package="FLASH-8-BRIDGE1" value="FLASH-BRIDGE1" x="47.2" y="-3.9"/>
-<element name="U$1" library="_openSX70" package="FLASH-8-BRIDGE-SW1-SW2-LED" value="FLASH-BRIDGE-SW1-SW2-LED" x="47.2" y="-0.3"/>
+<element name="U$2" library="_openSX70" library_urn="urn:adsk.eagle:library:7902803" package="FLASH-8-BRIDGE1" package3d_urn="urn:adsk.eagle:package:7902947/1" value="FLASH-BRIDGE1" x="47.2" y="-3.9"/>
+<element name="U$1" library="_openSX70" library_urn="urn:adsk.eagle:library:7902803" package="FLASH-8-BRIDGE-SW1-SW2-LED" package3d_urn="urn:adsk.eagle:package:7902948/1" value="FLASH-BRIDGE-SW1-SW2-LED" x="47.2" y="-0.3"/>
 </elements>
 <signals>
@@
 </note>
 <note version="8.3" severity="warning">
+Since Version 8.3, EAGLE supports Fusion synchronisation.
+This feature will not be available in this version and saving
+the document will break the link to the Fusion PCB feature.
+</note>
+<note version="8.3" severity="warning">
