File: 20190105_ORIGAMI_V1-H-08slot.sch (EAGLE design)
At the start: 21 parts, among them X1 JACK-SMD-SJ-3523-SMT-TR

Commit message: chanmges
Parts:
- DS2408: device DS2408-joaco:DS2408 -> _openSX70:DS2408
- OPTO: device openSX70:TLP127 -> _openSX70:TLP127
Changed lines of the file:
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@@
 </classes>
 <parts>
-<part name="DS2408" library="DS2408-joaco" deviceset="DS2408" device=""/>
+<part name="DS2408" library="_openSX70" library_urn="urn:adsk.eagle:library:7902803" deviceset="DS2408" device="" package3d_urn="urn:adsk.eagle:package:7902916/2"/>
 <part name="R1" library="Seeed-Resistor" library_urn="urn:adsk.eagle:library:474" deviceset="SMD-RES-4.7K-5%-1/10W(0603)" device="" package3d_urn="urn:adsk.eagle:package:32791/1" value="4.7K"/>
 <part name="R2" library="Seeed-Resistor" library_urn="urn:adsk.eagle:library:474" deviceset="SMD-RES-100K-1%-1/10W(0603)" device="" package3d_urn="urn:adsk.eagle:package:32791/1" value="100K"/>
@@
 <part name="R8" library="Seeed-Resistor" library_urn="urn:adsk.eagle:library:474" deviceset="SMD-RES-100K-1%-1/10W(0603)" device="" package3d_urn="urn:adsk.eagle:package:32791/1" value="100K"/>
 <part name="R9" library="Seeed-Resistor" library_urn="urn:adsk.eagle:library:474" deviceset="SMD-RES-220R-5%-1/10W(0603)" device="" package3d_urn="urn:adsk.eagle:package:32791/1" value="220R"/>
-<part name="SELECTOR" library="_openSX70" deviceset="SELECTOR-4-1-SMD-A6RS" device=""/>
+<part name="SELECTOR" library="_openSX70" library_urn="urn:adsk.eagle:library:7902803" deviceset="SELECTOR-4-1-SMD-A6RS" device="" package3d_urn="urn:adsk.eagle:package:7902943/4"/>
 <part name="LED1" library="SparkFun-LED" library_urn="urn:adsk.eagle:library:529" deviceset="LED-YELLOW" device="LILYPAD" package3d_urn="urn:adsk.eagle:package:39352/1" value="Yellow"/>
-<part name="OPTO" library="openSX70" deviceset="TLP127" device="" value="TLP127"/>
+<part name="OPTO" library="_openSX70" library_urn="urn:adsk.eagle:library:7902803" deviceset="TLP127" device="" package3d_urn="urn:adsk.eagle:package:7902924/3" value="TLP127"/>
 <part name="R12" library="Seeed-Resistor" library_urn="urn:adsk.eagle:library:474" deviceset="SMD-RES-220R-5%-1/10W(0603)" device="" package3d_urn="urn:adsk.eagle:package:32791/1" value="220R"/>
 <part name="FRAME1" library="frames" library_urn="urn:adsk.eagle:library:229" deviceset="DINA4_L" device=""/>
@@
 <part name="C1" library="Seeed-Capacitor" library_urn="urn:adsk.eagle:library:464" deviceset="CERAMIC-1UF-25V-10%-X7R(0603)" device="" package3d_urn="urn:adsk.eagle:package:32378/1" value="1uf"/>
 <part name="C2" library="Seeed-Capacitor" library_urn="urn:adsk.eagle:library:464" deviceset="CERAMIC-1UF-25V-10%-X7R(0603)" device="" package3d_urn="urn:adsk.eagle:package:32378/1" value="1uf"/>
-<part name="X1" library="_openSX70" deviceset="JACK-SMD-SJ-3523-SMT-TR" device=""/>
-<part name="U$2" library="_openSX70" deviceset="FLASH-BRIDGE1" device=""/>
-<part name="U$1" library="_openSX70" deviceset="FLASH-BRIDGE-SW1-SW2-LED" device=""/>
+<part name="X1" library="_openSX70" library_urn="urn:adsk.eagle:library:7902803" deviceset="JACK-SMD-SJ-3523-SMT-TR" device="" package3d_urn="urn:adsk.eagle:package:7902944/3"/>
+<part name="U$2" library="_openSX70" library_urn="urn:adsk.eagle:library:7902803" deviceset="FLASH-BRIDGE1" device="" package3d_urn="urn:adsk.eagle:package:7902947/1"/>
+<part name="U$1" library="_openSX70" library_urn="urn:adsk.eagle:library:7902803" deviceset="FLASH-BRIDGE-SW1-SW2-LED" device="" package3d_urn="urn:adsk.eagle:package:7902948/1"/>
 </parts>
 <sheets>
