File: 20190105_ORIGAMI_V1-V-2.brd (EAGLE design)
At the start: 32.7 x 12.1 mm, 5 parts, among them SW1 MK-12C02 G1.5, SW2 MK-12C02 G1.5

Commit message: 3D parts
Routing:
- net N$5: track 12.2 -> 0.00 mm
- net 2.8V-V: track 28.9 -> 18.4 mm, vias 2 -> 1
- net N$2: track 23.1 -> 18.1 mm, vias 0 -> 1
- net N$1: track 6.02 -> 8.75 mm
- net N$4: track 11.1 -> 9.57 mm
Changed lines of the file:
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@@
 <contactref element="U$1" pad="VCC-2.8V"/>
 <contactref element="LED" pad="A"/>
+<wire x1="23.3172" y1="11.2014" x2="23.2172" y2="11.2014" width="0.3048" layer="1"/>
+<wire x1="23.2172" y1="11.2014" x2="22.570953125" y2="11.847646875" width="0.3048" layer="1"/>
+<wire x1="24.746" y1="11.2014" x2="23.3172" y2="11.2014" width="0.3048" layer="16"/>
+<wire x1="27.4892" y1="8.4582" x2="24.746" y2="11.2014" width="0.3048" layer="16"/>
+<wire x1="29.2608" y1="8.4582" x2="27.4892" y2="8.4582" width="0.3048" layer="16"/>
+<wire x1="22.570953125" y1="11.847646875" x2="22.35" y2="12.2" width="0.3048" layer="1"/>
+<wire x1="29.2608" y1="8.4582" x2="29.45" y2="8.34" width="0.3048" layer="16"/>
+<wire x1="22.1742" y1="12.1158" x2="19.6596" y2="12.1158" width="0.3048" layer="1"/>
+<wire x1="22.1742" y1="12.1158" x2="22.35" y2="12.2" width="0.3048" layer="1"/>
+<wire x1="33.147" y1="7.3152" x2="35.10095" y2="9.26915" width="0.3048" layer="16"/>
+<wire x1="30.4038" y1="7.3152" x2="33.147" y2="7.3152" width="0.3048" layer="16"/>
+<wire x1="29.4894" y1="8.2296" x2="30.4038" y2="7.3152" width="0.3048" layer="16"/>
+<wire x1="29.4894" y1="8.2296" x2="29.45" y2="8.34" width="0.3048" layer="16"/>
+<via x="23.3172" y="11.2014" extent="1-16" drill="0.3048"/>
 <contactref element="SW2" pad="1"/>
 <contactref element="SW1" pad="1"/>
-<wire x1="25" y1="9.5" x2="22.5" y2="12" width="0.3048" layer="1"/>
-<wire x1="28" y1="9.5" x2="25" y2="9.5" width="0.3048" layer="1"/>
-<wire x1="29" y1="8.5" x2="28" y2="9.5" width="0.3048" layer="16"/>
-<wire x1="22.5" y1="12" x2="22.35" y2="12.2" width="0.3048" layer="1"/>
-<wire x1="29" y1="8.5" x2="29.45" y2="8.34" width="0.3048" layer="16"/>
-<wire x1="13" y1="10" x2="11" y2="10" width="0.3048" layer="16"/>
-<wire x1="16.5" y1="10" x2="13" y2="10" width="0.3048" layer="1"/>
-<wire x1="18.5" y1="12" x2="16.5" y2="10" width="0.3048" layer="1"/>
-<wire x1="22" y1="12" x2="18.5" y2="12" width="0.3048" layer="1"/>
-<wire x1="11" y1="10" x2="11.085" y2="9.74" width="0.3048" layer="16"/>
-<wire x1="22" y1="12" x2="22.35" y2="12.2" width="0.3048" layer="1"/>
-<wire x1="28" y1="9.5" x2="35.5" y2="9.5" width="0.3048" layer="16"/>
-<wire x1="35.5" y1="9.5" x2="35.585" y2="9.74" width="0.3048" layer="16"/>
-<via x="28" y="9.5" extent="1-16" drill="0.3048"/>
-<via x="13" y="10" extent="1-16" drill="0.3048"/>
+<wire x1="35.10095" y1="9.26915" x2="35.585" y2="9.74" width="0" layer="19" extent="16-16"/>
+<wire x1="11.085" y1="9.74" x2="19.6596" y2="12.1158" width="0" layer="19" extent="1-16"/>
 </signal>
 <signal name="N$1">
 <contactref element="U$2" pad="GND"/>
 <contactref element="U$1" pad="GND"/>
-<wire x1="17" y1="9.5" x2="17" y2="8.5" width="0.3048" layer="16"/>
-<wire x1="17" y1="5.5" x2="17" y2="9.5" width="0.3048" layer="1"/>
-<wire x1="17" y1="8.5" x2="17.2096" y2="8.1622" width="0.3048" layer="16"/>
-<wire x1="17" y1="5.5" x2="16.61" y2="5.011" width="0.3048" layer="1"/>
-<via x="17" y="9.5" extent="1-16" drill="0.3048"/>
+<wire x1="17.3736" y1="8.9154" x2="17.3736" y2="8.2296" width="0.3048" layer="16"/>
+<wire x1="18.6594" y1="10.2012" x2="17.3736" y2="8.9154" width="0.3048" layer="16"/>
+<wire x1="18.6594" y1="10.2012" x2="16.6878" y2="8.2296" width="0.3048" layer="1"/>
+<wire x1="16.6878" y1="5.0292" x2="16.6878" y2="8.2296" width="0.3048" layer="1"/>
+<wire x1="17.3736" y1="8.2296" x2="17.2096" y2="8.1622" width="0.3048" layer="16"/>
+<wire x1="16.6878" y1="5.0292" x2="16.61" y2="5.011" width="0.3048" layer="1"/>
+<via x="18.6594" y="10.2012" extent="1-16" drill="0.3048"/>
 </signal>
 <signal name="N$4">
 <contactref element="U$1" pad="LED"/>
 <contactref element="LED" pad="C"/>
-<wire x1="26" y1="10.5" x2="24.5" y2="12" width="0.3048" layer="1"/>
-<wire x1="28" y1="8.5" x2="26" y2="10.5" width="0.3048" layer="16"/>
-<wire x1="28" y1="7.5" x2="28" y2="8.5" width="0.3048" layer="16"/>
-<wire x1="28.5" y1="7" x2="28" y2="7.5" width="0.3048" layer="16"/>
-<wire x1="31" y1="7" x2="28.5" y2="7" width="0.3048" layer="16"/>
-<wire x1="32" y1="8" x2="31" y2="7" width="0.3048" layer="16"/>
-<wire x1="24.5" y1="12" x2="24.45" y2="12.2" width="0.3048" layer="1"/>
-<wire x1="32" y1="8" x2="32.02" y2="8.34" width="0.3048" layer="16"/>
-<via x="26" y="10.5" extent="1-16" drill="0.3048"/>
+<wire x1="25.546" y1="12.1158" x2="24.4602" y2="12.1158" width="0.3048" layer="1"/>
+<wire x1="26.0604" y1="11.2014" x2="26.0604" y2="11.6014" width="0.3048" layer="1"/>
+<wire x1="26.0604" y1="11.6014" x2="25.546" y2="12.1158" width="0.3048" layer="1"/>
+<wire x1="26.1034" y1="11.1584" x2="26.0604" y2="11.2014" width="0.3048" layer="16"/>
+<wire x1="26.1034" y1="11.1584" x2="26.1034" y2="11.0298" width="0.3048" layer="16"/>
+<wire x1="27.0606" y1="10.0726" x2="26.1034" y2="11.0298" width="0.3048" layer="16"/>
+<wire x1="30.3896" y1="10.0726" x2="27.0606" y2="10.0726" width="0.3048" layer="16"/>
+<wire x1="32.004" y1="8.4582" x2="30.3896" y2="10.0726" width="0.3048" layer="16"/>
+<wire x1="24.4602" y1="12.1158" x2="24.45" y2="12.2" width="0.3048" layer="1"/>
+<wire x1="32.004" y1="8.4582" x2="32.02" y2="8.34" width="0.3048" layer="16"/>
+<via x="26.0604" y="11.2014" extent="1-16" drill="0.3048"/>
 </signal>
 <signal name="GND">
@@
 <contactref element="SW2" pad="2"/>
 <contactref element="U$1" pad="SWITCH-2"/>
-<wire x1="37.5" y1="8.5" x2="38.5" y2="9.5" width="0.3048" layer="16"/>
-<wire x1="34.5" y1="8.5" x2="37.5" y2="8.5" width="0.3048" layer="16"/>
-<wire x1="32.5" y1="6.5" x2="34.5" y2="8.5" width="0.3048" layer="16"/>
-<wire x1="28" y1="6.5" x2="32.5" y2="6.5" width="0.3048" layer="16"/>
-<wire x1="26" y1="8.5" x2="28" y2="6.5" width="0.3048" layer="16"/>
-<wire x1="26" y1="9.5" x2="26" y2="8.5" width="0.3048" layer="16"/>
-<wire x1="20.5" y1="9.5" x2="26" y2="9.5" width="0.3048" layer="16"/>
-<wire x1="19.5" y1="8.5" x2="20.5" y2="9.5" width="0.3048" layer="16"/>
-<wire x1="38.5" y1="9.5" x2="38.585" y2="9.74" width="0.3048" layer="16"/>
-<wire x1="19.5" y1="8.5" x2="19.17" y2="8.34" width="0.3048" layer="16"/>
+<wire x1="21.2598" y1="10.5156" x2="36.3474" y2="10.5156" width="0.3048" layer="1"/>
+<wire x1="19.2024" y1="8.4582" x2="21.2598" y2="10.5156" width="0.3048" layer="16"/>
+<wire x1="19.2024" y1="8.4582" x2="19.17" y2="8.34" width="0.3048" layer="16"/>
+<via x="21.2598" y="10.5156" extent="1-16" drill="0.3048"/>
+<wire x1="36.3474" y1="10.5156" x2="38.585" y2="9.74" width="0" layer="19" extent="1-16"/>
 </signal>
 <signal name="N$5">
 <contactref element="SW1" pad="2"/>
 <contactref element="U$1" pad="SWITCH-1"/>
-<wire x1="15" y1="8.5" x2="14" y2="9.5" width="0.3048" layer="16"/>
-<wire x1="15.5" y1="8.5" x2="15" y2="8.5" width="0.3048" layer="16"/>
-<wire x1="17" y1="7" x2="15.5" y2="8.5" width="0.3048" layer="16"/>
-<wire x1="23" y1="7" x2="17" y2="7" width="0.3048" layer="16"/>
-<wire x1="24" y1="8" x2="23" y2="7" width="0.3048" layer="16"/>
-<wire x1="14" y1="9.5" x2="14.085" y2="9.74" width="0.3048" layer="16"/>
-<wire x1="24" y1="8" x2="24.31" y2="8.34" width="0.3048" layer="16"/>
+<wire x1="14.085" y1="9.74" x2="24.31" y2="8.34" width="0" layer="19" extent="16-16"/>
 </signal>
 </signals>
