File: origami/20190105_ORIGAMI_V1-V-3.sch (EAGLE design)
At the start: 5 parts, among them SW1 MK-12C02 G1.5, SW2 MK-12C02 G1.5

Commit message: I am confused, hopefully this works
Parts:
- U$1: value FLASH-BRIDGE-SW1-SW2-LED-SMALL -> FLASH-BRIDGE-SW1-SW2-LED-SMALL-NO-GND; device _openSX70:FLASH-BRIDGE-SW1-SW2-LED-SMALL -> _openSX70:FLASH-BRIDGE-SW1-SW2-LED-SMALL-NO-GND
Connections:
- net N$1: no longer U$1.GND
Changed lines of the file:
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@@
 <?xml version="1.0" encoding="utf-8"?>
 <!DOCTYPE eagle SYSTEM "eagle.dtd">
-<eagle version="9.2.0">
+<eagle version="9.2.2">
 <drawing>
 <settings>
@@
 <part name="SW1" library="_openSX70" library_urn="urn:adsk.eagle:library:7902803" deviceset="K3-1280S-SHORT" device="SMALL" value="MK-12C02 G1.5"/>
 <part name="SW2" library="_openSX70" library_urn="urn:adsk.eagle:library:7902803" deviceset="K3-1280S-SHORT" device="SMALL" value="MK-12C02 G1.5"/>
-<part name="U$1" library="_openSX70" library_urn="urn:adsk.eagle:library:7902803" deviceset="FLASH-BRIDGE-SW1-SW2-LED-SMALL" device="" package3d_urn="urn:adsk.eagle:package:7902950/1"/>
+<part name="U$1" library="_openSX70" library_urn="urn:adsk.eagle:library:7902803" deviceset="FLASH-BRIDGE-SW1-SW2-LED-SMALL-NO-GND" device=""/>
 <part name="U$2" library="_openSX70" library_urn="urn:adsk.eagle:library:7902803" deviceset="SX70-FLASH-EDGE8-MALE-LONG" device="" package3d_urn="urn:adsk.eagle:package:7902946/1"/>
 <part name="LED" library="led" library_urn="urn:adsk.eagle:library:259" deviceset="LED" device="CHIP-LED0805" package3d_urn="urn:adsk.eagle:package:15818/2"/>
@@
 </plain>
 <instances>
-<instance part="FRAME1" gate="G$1" x="-7.62" y="-15.24"/>
-<instance part="FRAME1" gate="G$2" x="154.94" y="-15.24">
+<instance part="FRAME1" gate="G$1" x="-7.62" y="-15.24" smashed="yes"/>
+<instance part="FRAME1" gate="G$2" x="154.94" y="-15.24" smashed="yes">
 <attribute name="LAST_DATE_TIME" x="167.64" y="-13.97" size="2.54" layer="94"/>
 <attribute name="SHEET" x="241.3" y="-13.97" size="2.54" layer="94"/>
 <attribute name="DRAWING_NAME" x="172.72" y="3.81" size="2.54" layer="94"/>
 </instance>
-<instance part="SW1" gate="G$1" x="187.96" y="78.74" rot="R180">
+<instance part="SW1" gate="G$1" x="187.96" y="78.74" smashed="yes" rot="R180">
 <attribute name="NAME" x="195.58" y="85.09" size="1.27" layer="95" ratio="10" rot="R270"/>
 </instance>
-<instance part="SW2" gate="G$1" x="187.96" y="101.6" rot="R180">
+<instance part="SW2" gate="G$1" x="187.96" y="101.6" smashed="yes" rot="R180">
 <attribute name="NAME" x="195.58" y="107.95" size="1.27" layer="95" ratio="10" rot="R270"/>
 </instance>
-<instance part="U$1" gate="G$1" x="109.22" y="78.74" rot="R270"/>
-<instance part="U$2" gate="G$1" x="109.22" y="33.02" rot="R270"/>
-<instance part="LED" gate="G$1" x="129.54" y="60.96" rot="R270">
+<instance part="U$1" gate="G$1" x="109.22" y="78.74" smashed="yes" rot="R270"/>
+<instance part="U$2" gate="G$1" x="109.22" y="33.02" smashed="yes" rot="R270"/>
+<instance part="LED" gate="G$1" x="129.54" y="60.96" smashed="yes" rot="R270">
 <attribute name="NAME" x="124.968" y="57.404" size="1.778" layer="95"/>
 <attribute name="VALUE" x="124.968" y="55.245" size="1.778" layer="96"/>
@@
 <pinref part="U$2" gate="G$1" pin="GND"/>
 <wire x1="137.16" y1="50.8" x2="119.38" y2="50.8" width="0.1524" layer="91"/>
-<pinref part="U$1" gate="G$1" pin="GND"/>
-<wire x1="119.38" y1="96.52" x2="137.16" y2="96.52" width="0.1524" layer="91"/>
-<wire x1="137.16" y1="96.52" x2="137.16" y2="50.8" width="0.1524" layer="91"/>
 </segment>
 </net>
