File: PUSH/PCBWAY/openSX70-dongle_v6-2-dual-led.brd (EAGLE design)
At the start: 160 x 100 mm, 21 parts, among them J1 MJ1-2503A

Commit message: NEW DUAL LED
Other:
- board size 160 x 100 mm -> 40.6 x 30.5 mm
