File: PUSH/PCBWAY/openSX70-dongle_v6-3-dual-led.brd (EAGLE design)
At the start: 160 x 100 mm, 21 parts, among them J1 MJ1-2503A

Commit message: NEW DUAL LED
Other:
- board size 160 x 100 mm -> 40.6 x 30.5 mm
- board text added: "1000"
- board text added: "130"
- board text added: "20"
- board text added: "2000"
- board text added: "25"
- board text added: "260"
- board text added: "30"
- board text added: "4"
- board text added: "45"
- board text added: "500"
- board text added: "60"
- board text added: "8"
- board text added: "uDongle 6.3 20190515"
- board text removed: "EV10"
- board text removed: "EV10.5"
- board text removed: "EV11"
- board text removed: "EV11.5"
- board text removed: "EV12"
- board text removed: "EV13"
- board text removed: "EV14"
- board text removed: "EV15"
- board text removed: "EV16"
- board text removed: "EV17"
- board text removed: "EV8"
- board text removed: "EV9"
- board text removed: "uDongle 6.2 20190515"
